Commit message: finish static desk avoid

File: src/ocs2_tracer_jaka/tracer_jaka_mujoco/urdf/tracer_jaka_zu5_real.urdf (robot description, URDF)
Before this commit: robot tracer_jaka_zu5, 31 links, 30 joints
Links:
- link Link_0: geometry collision sphere radius=0.085; visual mesh filename=package://tracer_jaka_mujoco/urdf/meshes/Link_0.STL
- link Link_1: geometry collision sphere radius=0.075; visual mesh filename=package://tracer_jaka_mujoco/urdf/meshes/Link_1.STL
- link Link_2: geometry collision sphere radius=0.065; collision sphere radius=0.065
- link Link_3: geometry collision sphere radius=0.05; collision sphere radius=0.05
- link Link_4: geometry collision sphere radius=0.05; visual mesh filename=package://tracer_jaka_mujoco/urdf/meshes/Link_4.STL
- link Link_5: geometry collision sphere radius=0.05; visual mesh filename=package://tracer_jaka_mujoco/urdf/meshes/Link_5.STL
- link Link_6: geometry collision sphere radius=0.045; visual mesh filename=package://tracer_jaka_mujoco/urdf/meshes/Link_6.STL
- link base_link: geometry collision sphere radius=0.17; collision sphere radius=0.17
- link d435i_link: geometry collision sphere radius=0.035; visual mesh filename=package://tracer_jaka_mujoco/urdf/meshes/realsense_d435.stl
- link fl_wheel_link: geometry visual mesh filename=package://tracer_jaka_mujoco/urdf/meshes/castor.dae
- link fr_wheel_link: geometry visual mesh filename=package://tracer_jaka_mujoco/urdf/meshes/castor.dae
- link left_wheel_link: geometry visual mesh filename=package://tracer_jaka_mujoco/urdf/meshes/tracer_wheel.dae
- link right_wheel_link: geometry visual mesh filename=package://tracer_jaka_mujoco/urdf/meshes/tracer_wheel.dae
- link rl_wheel_link: geometry visual mesh filename=package://tracer_jaka_mujoco/urdf/meshes/castor.dae
- link rr_wheel_link: geometry visual mesh filename=package://tracer_jaka_mujoco/urdf/meshes/castor.dae
- link tool0_and_camera_link: geometry collision sphere radius=0.045; collision sphere radius=0.045
- link urbase_base_link: geometry visual mesh filename=package://tracer_jaka_mujoco/urdf/meshes/urbase_base_link.S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
Joints:
- joint left_wheel: axis 0 1 0 -> (none); limit effort=50 velocity=10 -> (none); type continuous -> fixed
- joint right_wheel: axis 0 1 0 -> (none); limit effort=50 velocity=10 -> (none); type continuous -> fixed
- joint tool0_and_camera_link_joint: origin xyz=0 0 0 rpy=0 0 -2.3561945 -> xyz=0 0 0 rpy=0 0 -0.7853
